File: BatteryEmulator - WIFI/BatteryEmulator.kicad_sch (KiCad schematic)
At the start: 211 parts, among them J1 Barrel_Jack_MountingPin, J2 Barrel_Jack_Switch_MountingPin, J3 Conn_01x16, J4 Conn_01x08, U1 AMS1117CD-5.0, U10 TMR_1-0513, U11 AMS1117CD-5.0, U12 AMS1117CD-5.0, U13 TMR_1-0513, U14 TMR_1-0513, U15 AMS1117CD-5.0, U16 AMS1117CD-5.0, U17 TMR_1-0513, U18 TMR_1-0513, U19 TMR_1-0513, U2 TMR_1-0513, U20 TMR_1-0513, U21 AMS1117CD-5.0, U22 AMS1117CD-5.0, U23 AMS1117CD-5.0, U24 AMS1117CD-5.0, U25 TMR_1-0513, U26 TMR_1-0513, U27 AMS1117CD-5.0, U28 TMR_1-0513, U29 AMS1117CD-5.0, U3 TMR_1-0513, U30 AMS1117CD-5.0, U31 AMS1117CD-5.0, U33 TMR_1-0513, U34 TMR_1-0513, U35 AMS1117CD-5.0, U4 AMS1117CD-5.0, U5 TMR_1-0513, U6 TMR_1-0513, U7 AMS1117CD-5.0, U8 AMS1117CD-5.0

Commit message: Complete Schematics of analog version
Parts:
- removed C65: C_0805, Capacitor_SMD:C_0805_2012Metric, symbol PCM_Capacitor_AKL:C_0805
- removed D1: LED, symbol Device:LED
- removed D2: D_Schottky, symbol Device:D_Schottky
- removed F2: Fuse, symbol Device:Fuse
- removed J2: Barrel_Jack_Switch_MountingPin, symbol Connector:Barrel_Jack_Switch_MountingPin
- removed J3: Conn_01x16, symbol Connector_Generic:Conn_01x16
- removed J4: Conn_01x08, symbol Connector_Generic:Conn_01x08
- removed R39: R_0805, Resistor_SMD:R_0805_2012Metric, symbol PCM_Resistor_AKL:R_0805
- removed RV17, RV19, RV20, RV21, RV22, RV23, RV24, RV25, RV26, RV27, RV28, RV29, RV30, RV31, RV32, RV33, RV34: R_Potentiometer_US, Potentiometer_THT:Potentiometer_Alps_RK09Y11_Single_Horizontal, symbol Device:R_Potentiometer_US
