File: BatteryEmulator/BatteryEmulator.kicad_sch (KiCad schematic)
At the start: 211 parts, among them J1 Barrel_Jack_MountingPin, J2 Barrel_Jack_Switch_MountingPin, J3 Conn_01x16, J4 Conn_01x08, U1 AMS1117CD-5.0, U10 TMR_1-0513, U11 AMS1117CD-5.0, U12 AMS1117CD-5.0, U13 TMR_1-0513, U14 TMR_1-0513, U15 AMS1117CD-5.0, U16 AMS1117CD-5.0, U17 TMR_1-0513, U18 TMR_1-0513, U19 TMR_1-0513, U2 TMR_1-0513, U20 TMR_1-0513, U21 AMS1117CD-5.0, U22 AMS1117CD-5.0, U23 AMS1117CD-5.0, U24 AMS1117CD-5.0, U25 TMR_1-0513, U26 TMR_1-0513, U27 AMS1117CD-5.0, U28 TMR_1-0513, U29 AMS1117CD-5.0, U3 TMR_1-0513, U30 AMS1117CD-5.0, U31 AMS1117CD-5.0, U33 TMR_1-0513, U34 TMR_1-0513, U35 AMS1117CD-5.0, U4 AMS1117CD-5.0, U5 TMR_1-0513, U6 TMR_1-0513, U7 AMS1117CD-5.0, U8 AMS1117CD-5.0

Commit message: Backup
Parts:
- removed J2: Barrel_Jack_Switch_MountingPin, symbol Connector:Barrel_Jack_Switch_MountingPin
- added J2: Barrel_Jack_MountingPin, Connector_Molex:Molex_KK-396_5273-02A_1x02_P3.96mm_Vertical, symbol Connector:Barrel_Jack_MountingPin
- added J5: Barrel_2.0mmPin_PJ064, Connector_BarrelJack:BarrelJack_GCT_DCJ200-10-A_Horizontal, symbol PCM_4ms_Jack:Barrel_2.0mmPin_PJ064
- D1: footprint (none) -> LED_THT:LED_D3.0mm
- D2, F1, F2: footprint (none) -> Resistor_SMD:R_1206_3216Metric
- J1: footprint (none) -> Connector_Molex:Molex_KK-396_5273-02A_1x02_P3.96mm_Vertical
- J3: footprint (none) -> Connector_PinHeader_2.54mm:PinHeader_1x16_P2.54mm_Vertical
- J4: footprint (none) -> Connector_PinHeader_2.54mm:PinHeader_1x08_P2.54mm_Vertical
Connections:
- net CTREF: now also J2.1, J2.2
- net GND: now also J5.2
- net at F2.1: now also J5.1
Changed lines of the file:
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@@
   (junction (at 127 138.43) (diameter 0) (color 0 0 0 0)
   )
-  (junction (at 463.55 121.92) (diameter 0) (color 0 0 0 0)
-  )
   (junction (at 248.92 278.13) (diameter 0) (color 0 0 0 0)
   )
@@
   (junction (at 118.11 336.55) (diameter 0) (color 0 0 0 0)
   )
+  (junction (at 464.82 59.69) (diameter 0) (color 0 0 0 0)
+  )
   (junction (at 36.83 36.83) (diameter 0) (color 0 0 0 0)
   )
@@
   (junction (at 207.01 184.15) (diameter 0) (color 0 0 0 0)
   )
-  (junction (at 466.09 116.84) (diameter 0) (color 0 0 0 0)
-  )
   (junction (at 255.27 368.3) (diameter 0) (color 0 0 0 0)
   )
@@
     (stroke (width 0) (type default))
   )
+  (wire (pts (xy 466.09 116.84) (xy 466.09 121.92))
+    (stroke (width 0) (type default))
+  )
   (wire (pts (xy 127 95.25) (xy 130.81 95.25))
     (stroke (width 0) (type default))
@@
     (stroke (width 0) (type default))
   )
-  (wire (pts (xy 466.09 116.84) (xy 466.09 121.92))
-    (stroke (width 0) (type default))
-  )
   (wire (pts (xy 245.11 355.6) (xy 255.27 355.6))
     (stroke (width 0) (type default))
@@
     (stroke (width 0) (type default))
   )
-  (wire (pts (xy 466.09 114.3) (xy 466.09 116.84))
-    (stroke (width 0) (type default))
-  )
   (wire (pts (xy 36.83 317.5) (xy 36.83 311.15))
     (stroke (width 0) (type default))
@@
     (stroke (width 0) (type default))
   )
+  (wire (pts (xy 464.82 59.69) (xy 464.82 62.23))
+    (stroke (width 0) (type default))
+  )
   (wire (pts (xy 36.83 302.26) (xy 36.83 300.99))
     (stroke (width 0) (type default))
@@
     (stroke (width 0) (type default))
   )
+  (wire (pts (xy 464.82 59.69) (xy 474.98 59.69))
+    (stroke (width 0) (type default))
+  )
   (wire (pts (xy 199.39 90.17) (xy 199.39 96.52))
     (stroke (width 0) (type default))
@@
     (stroke (width 0) (type default))
   )
+  (wire (pts (xy 464.82 57.15) (xy 464.82 59.69))
+    (stroke (width 0) (type default))
+  )
   (wire (pts (xy 191.77 306.07) (xy 194.31 306.07))
     (stroke (width 0) (type default))
@@
     (stroke (width 0) (type default))
   )
-  (wire (pts (xy 458.47 121.92) (xy 463.55 121.92))
-    (stroke (width 0) (type default))
-  )
   (wire (pts (xy 36.83 78.74) (xy 36.83 71.12))
     (stroke (width 0) (type default))
@@
     )
   )
+  (global_label "TERMN" (shape output) (at 474.98 59.69 0) (fields_autoplaced)
+    (effects (font (size 1.27 1.27)) (justify left))
+    (property "Intersheetrefs" "${INTERSHEET_REFS}" (at 484.1337 59.69 0)
+      (effects (font (size 1.27 1.27)) (justify left) hide)
+    )
+  )
   (global_label "TERMP" (shape output) (at 492.76 85.09 0) (fields_autoplaced)
     (effects (font (size 1.27 1.27)) (justify left))
@@
       (effects (font (size 1.27 1.27)))
     )
-    (property "Footprint" "" (at 459.74 86.106 0)
+    (property "Footprint" "Connector_Molex:Molex_KK-396_5273-02A_1x02_P3.96mm_Vertical" (at 459.74 86.106 0)
       (effects (font (size 1.27 1.27)) hide)
     )
@@
     (pin "1")
     (pin "2")
-    (pin "4")
-    (pin "3")
     (pin "8")
+    (pin "3")
+    (pin "4")
     (instances
       (project "BatteryEmulator"
@@
     )
   )
+  (symbol (lib_id "PCM_4ms_Jack:Barrel_2.0mmPin_PJ064") (at 458.47 114.3 0) (unit 1)
+    (in_bom yes) (on_board yes) (dnp no) (fields_autoplaced)
+    (property "Reference" "J5" (at 458.47 105.41 0)
+      (effects (font (size 1.27 1.27)))
+    )
+    (property "Value" "Barrel_2.0mmPin_PJ064" (at 458.47 107.95 0)
+      (effects (font (size 1.27 1.27)))
+    )
+    (property "Footprint" "Connector_BarrelJack:BarrelJack_GCT_DCJ200-10-A_Horizontal" (at 458.851 107.442 0)
+      (effects (font (size 1.27 1.27)) hide)
+    )
+    (property "Datasheet" "" (at 459.74 115.316 0)
+      (effects (font (size 1.27 1.27)) hide)
+    )
+    (property "Specifications" "Barrel Jack, 2.0mm diameter center pin, Vertical, PC-pins" (at 455.93 122.174 0)
+      (effects (font (size 1.27 1.27)) (justify left) hide)
+    )
+    (property "Manufacturer" "Wenzhou QingPu Electronics Co" (at 455.93 123.698 0)
+      (effects (font (size 1.27 1.27)) (justify left) hide)
+    )
+    (property "Part Number" "WQP-DC026M (2.0mm center pin)" (at 455.93 125.222 0)
+      (effects (font (size 1.27 1.27)) (justify left) hide)
+    )
+    (pin "1")
+    (pin "2")
+    (pin "3")
+    (instances
+      (project "BatteryEmulator"
+        (path "/f36eed8c-9d65-456e-bb95-b77a2c4a1b89"
+          (reference "J5") (unit 1)
+        )
+      )
+    )
+  )
   (symbol (lib_id "Converter_DCDC:ITX4805SA") (at 54.61 41.91 0) (unit 1)
     (in_bom yes) (on_board yes) (dnp no) (fields_autoplaced)
@@
       (effects (font (size 1.27 1.27)) (justify right))
     )
-    (property "Footprint" "" (at 505.46 115.57 0)
+    (property "Footprint" "LED_THT:LED_D3.0mm" (at 505.46 115.57 0)
       (effects (font (size 1.27 1.27)) hide)
     )
@@
       (effects (font (size 1.27 1.27)))
     )
-    (property "Footprint" "" (at 485.14 111.76 0)
+    (property "Footprint" "Resistor_SMD:R_1206_3216Metric" (at 485.14 111.76 0)
       (effects (font (size 1.27 1.27)) hide)
     )
@@
     )
   )
+  (symbol (lib_id "Connector:Barrel_Jack_MountingPin") (at 457.2 59.69 0) (unit 1)
+    (in_bom yes) (on_board yes) (dnp no) (fields_autoplaced)
+    (property "Reference" "J2" (at 457.2 50.8 0)
+      (effects (font (size 1.27 1.27)))
+    )
+    (property "Value" "Barrel_Jack_MountingPin" (at 457.2 53.34 0)
+      (effects (font (size 1.27 1.27)))
+    )
+    (property "Footprint" "Connector_Molex:Molex_KK-396_5273-02A_1x02_P3.96mm_Vertical" (at 458.47 60.706 0)
+      (effects (font (size 1.27 1.27)) hide)
+    )
+    (property "Datasheet" "~" (at 458.47 60.706 0)
+      (effects (font (size 1.27 1.27)) hide)
+    )
+    (pin "1")
+    (pin "2")
+    (pin "MP")
+    (instances
+      (project "BatteryEmulator"
+        (path "/f36eed8c-9d65-456e-bb95-b77a2c4a1b89"
+          (reference "J2") (unit 1)
+        )
+      )
+    )
+  )
   (symbol (lib_id "PCM_Capacitor_AKL:C_0805") (at 85.09 167.64 0) (unit 1)
     (in_bom yes) (on_board yes) (dnp no) (fields_autoplaced)
@@
       (effects (font (size 1.27 1.27)))
     )
-    (property "Footprint" "" (at 480.06 86.868 90)
+    (property "Footprint" "Resistor_SMD:R_1206_3216Metric" (at 480.06 86.868 90)
       (effects (font (size 1.27 1.27)) hide)
     )
@@
       (effects (font (size 1.27 1.27)) (justify left))
     )
-    (property "Footprint" "" (at 520.7 173.99 0)
+    (property "Footprint" "Connector_PinHeader_2.54mm:PinHeader_1x16_P2.54mm_Vertical" (at 520.7 173.99 0)
       (effects (font (size 1.27 1.27)) hide)
     )
@@
   )
   (symbol (lib_id "Regulator_Switching:TMR_1-0513") (at 181.61 129.54 0) (unit 1)
-    (in_bom yes) (on_board yes) (dnp no) (fields_autoplaced)
+    (in_bom yes) (on_board yes) (dnp no)
     (property "Reference" "U25" (at 181.61 116.84 0)
       (effects (font (size 1.27 1.27)))
@@
       (effects (font (size 1.27 1.27)) (justify left))
     )
-    (property "Footprint" "" (at 548.64 163.83 0)
+    (property "Footprint" "Connector_PinHeader_2.54mm:PinHeader_1x08_P2.54mm_Vertical" (at 548.64 163.83 0)
       (effects (font (size 1.27 1.27)) hide)
     )
@@
     )
   )
-  (symbol (lib_id "Connector:Barrel_Jack_Switch_MountingPin") (at 458.47 114.3 0) (unit 1)
-    (in_bom yes) (on_board yes) (dnp no) (fields_autoplaced)
-    (property "Reference" "J2" (at 458.47 105.41 0)
-      (effects (font (size 1.27 1.27)))
-    )
-    (property "Value" "Barrel_Jack_Switch_MountingPin" (at 458.47 107.95 0)
-      (effects (font (size 1.27 1.27)))
-    )
-    (property "Footprint" "" (at 459.74 115.316 0)
-      (effects (font (size 1.27 1.27)) hide)
-    )
-    (property "Datasheet" "~" (at 459.74 115.316 0)
-      (effects (font (size 1.27 1.27)) hide)
-    )
-    (pin "1")
-    (pin "2")
-    (pin "3")
-    (pin "MP")
-    (instances
-      (project "BatteryEmulator"
-        (path "/f36eed8c-9d65-456e-bb95-b77a2c4a1b89"
-          (reference "J2") (unit 1)
-        )
-      )
-    )
-  )
   (symbol (lib_id "Regulator_Switching:TMR_1-0513") (at 54.61 41.91 0) (unit 1)
     (in_bom yes) (on_board yes) (dnp no) (fields_autoplaced)
@@
       (effects (font (size 1.27 1.27)))
     )
-    (property "Footprint" "" (at 474.98 113.538 90)
+    (property "Footprint" "Resistor_SMD:R_1206_3216Metric" (at 474.98 113.538 90)
       (effects (font (size 1.27 1.27)) hide)
     )
