File: BatteryEmulator/BatteryEmulator.kicad_pcb (KiCad board)
At the start: 2 copper layers, 145 parts, among them U1 AMS1117CD-5.0, U10 TMR_1-0513, U11 AMS1117CD-5.0, U12 AMS1117CD-5.0, U13 TMR_1-0513, U14 TMR_1-0513, U15 AMS1117CD-5.0, U16 AMS1117CD-5.0, U17 TMR_1-0513, U18 TMR_1-0513, U19 TMR_1-0513, U2 TMR_1-0513, U20 TMR_1-0513, U21 AMS1117CD-5.0, U22 AMS1117CD-5.0, U23 AMS1117CD-5.0, U24 AMS1117CD-5.0, U25 TMR_1-0513, U26 TMR_1-0513, U27 TMR_1-0513, U28 TMR_1-0513, U29 AMS1117CD-5.0, U3 TMR_1-0513, U30 AMS1117CD-5.0, U31 AMS1117CD-5.0, U32 AMS1117CD-5.0, U4 AMS1117CD-5.0, U5 TMR_1-0513, U6 TMR_1-0513, U7 AMS1117CD-5.0, U8 AMS1117CD-5.0, U9 TMR_1-0513

Commit message: Complete Schematics of analog version
Parts:
- removed U32: AMS1117CD-5.0, Package_TO_SOT_SMD:TO-252-3_TabPin2
- removed U9: TMR_1-0513, Converter_DCDC:Converter_DCDC_TRACO_TMR-1-xxxx_Single_THT
- added C65: C_0805, Capacitor_SMD:C_0805_2012Metric, F.Cu at (122.9, 168.4)
- added C67: C_0805, Capacitor_SMD:C_0805_2012Metric, F.Cu at (122.9, 171.4)
- added C69: C_0805, Capacitor_SMD:C_0805_2012Metric, F.Cu at (122.9, 174.4)
- added PS1: ITX4805SA, Converter_DCDC:Converter_DCDC_Murata_CRE1xxxxxxSC_THT, F.Cu at (96.0, 118.1)
- added PS10: ITX4805SA, Converter_DCDC:Converter_DCDC_Murata_CRE1xxxxxxSC_THT, F.Cu at (111.5, 131.3)
- added PS11: ITX4805SA, Converter_DCDC:Converter_DCDC_Murata_CRE1xxxxxxSC_THT, F.Cu at (119.3, 131.3)
- added PS12: ITX4805SA, Converter_DCDC:Converter_DCDC_Murata_CRE1xxxxxxSC_THT, F.Cu at (127.0, 131.3)
- added PS13: ITX4805SA, Converter_DCDC:Converter_DCDC_Murata_CRE1xxxxxxSC_THT, F.Cu at (134.8, 131.3)
- added PS14: ITX4805SA, Converter_DCDC:Converter_DCDC_Murata_CRE1xxxxxxSC_THT, F.Cu at (96.0, 144.5)
- added PS15: ITX4805SA, Converter_DCDC:Converter_DCDC_Murata_CRE1xxxxxxSC_THT, F.Cu at (103.7, 144.5)
- added PS16: ITX4805SA, Converter_DCDC:Converter_DCDC_Murata_CRE1xxxxxxSC_THT, F.Cu at (111.5, 144.5)
- added PS17: ITX4805SA, Converter_DCDC:Converter_DCDC_Murata_CRE1xxxxxxSC_THT, F.Cu at (119.3, 144.5)
- added PS2: ITX4805SA, Converter_DCDC:Converter_DCDC_Murata_CRE1xxxxxxSC_THT, F.Cu at (103.7, 118.1)
- added PS4: ITX4805SA, Converter_DCDC:Converter_DCDC_Murata_CRE1xxxxxxSC_THT, F.Cu at (111.5, 118.1)
- added PS5: ITX4805SA, Converter_DCDC:Converter_DCDC_Murata_CRE1xxxxxxSC_THT, F.Cu at (119.3, 118.1)
- added PS6: ITX4805SA, Converter_DCDC:Converter_DCDC_Murata_CRE1xxxxxxSC_THT, F.Cu at (127.0, 118.1)
- added PS7: ITX4805SA, Converter_DCDC:Converter_DCDC_Murata_CRE1xxxxxxSC_THT, F.Cu at (134.8, 118.1)
- added PS8: ITX4805SA, Converter_DCDC:Converter_DCDC_Murata_CRE1xxxxxxSC_THT, F.Cu at (96.0, 131.3)
- added PS9: ITX4805SA, Converter_DCDC:Converter_DCDC_Murata_CRE1xxxxxxSC_THT, F.Cu at (103.7, 131.3)
- added R33: R_0805, Resistor_SMD:R_0805_2012Metric, F.Cu at (109.4, 201.2)
- added R34: R_0805, Resistor_SMD:R_0805_2012Metric, F.Cu at (109.4, 204.1)
- added R35: R_0805, Resistor_SMD:R_0805_2012Metric, F.Cu at (109.4, 207.1)
- added R36: R_0805, Resistor_SMD:R_0805_2012Metric, F.Cu at (109.4, 210.0)
- added R37: R_0805, Resistor_SMD:R_0805_2012Metric, F.Cu at (113.8, 186.4)
- added R38: R_0805, Resistor_SMD:R_0805_2012Metric, F.Cu at (113.8, 189.4)
- added R39: R_0805, Resistor_SMD:R_0805_2012Metric, F.Cu at (113.8, 192.3)
- added R41: R_0805, Resistor_SMD:R_0805_2012Metric, F.Cu at (113.8, 195.3)
- added R42: R_0805, Resistor_SMD:R_0805_2012Metric, F.Cu at (113.8, 198.2)
- added R43: R_0805, Resistor_SMD:R_0805_2012Metric, F.Cu at (113.8, 201.2)
- added R44: R_0805, Resistor_SMD:R_0805_2012Metric, F.Cu at (113.8, 204.1)
- added R45: R_0805, Resistor_SMD:R_0805_2012Metric, F.Cu at (113.8, 207.1)
- added R46: R_0805, Resistor_SMD:R_0805_2012Metric, F.Cu at (113.8, 210.0)
- added R47: R_0805, Resistor_SMD:R_0805_2012Metric, F.Cu at (118.2, 186.4)
- added R48: R_0805, Resistor_SMD:R_0805_2012Metric, F.Cu at (118.2, 189.4)
- added R49: R_0805, Resistor_SMD:R_0805_2012Metric, F.Cu at (118.2, 192.3)
- added R50: R_0805, Resistor_SMD:R_0805_2012Metric, F.Cu at (118.2, 195.3)
- added R51: R_0805, Resistor_SMD:R_0805_2012Metric, F.Cu at (118.2, 198.2)
- added R52: R_0805, Resistor_SMD:R_0805_2012Metric, F.Cu at (118.2, 201.2)
- added R53: R_0805, Resistor_SMD:R_0805_2012Metric, F.Cu at (118.2, 204.1)
- added R54: R_0805, Resistor_SMD:R_0805_2012Metric, F.Cu at (118.2, 207.1)
- added RV18: R_Potentiometer, PCM_Potentiometer_THT_AKL:Potentiometer_Bourns_PTA6043_Single_Slide, F.Cu at (18.7, 209.9)
- added U33: TMR_1-0513, Converter_DCDC:Converter_DCDC_TRACO_TMR-1-xxxx_Single_THT, F.Cu at (134.6, 33.6)
- added U34: TMR_1-0513, Converter_DCDC:Converter_DCDC_TRACO_TMR-1-xxxx_Single_THT, F.Cu at (134.6, 42.8)
- added U35: AMS1117CD-5.0, Package_TO_SOT_SMD:TO-252-3_TabPin2, F.Cu at (125.2, 103.2)
- R1, R2, U1, U11, U12, U15, U16, U21, U22, U23, U24, U29, U30, U31, U4, U7, U8: moved to F.Cu
- RV17: value R_Potentiometer_MountingPin -> R_Potentiometer_US; footprint PCM_Potentiometer_THT_AKL:Potentiometer_Bourns_PTA6043_Single_Slide -> Potentiometer_THT:Potentiometer_Alps_RK09Y11_Single_Horizontal
- U27: value TMR_1-0513 -> AMS1117CD-5.0; footprint Converter_DCDC:Converter_DCDC_TRACO_TMR-1-xxxx_Single_THT -> Package_TO_SOT_SMD:TO-252-3_TabPin2
- moved R32 240.9 mm to (109.4, 198.2)
- moved R28 238.9 mm to (109.4, 186.4)
- moved RV17 237.6 mm to (136.7, 188.0)
- moved C60 236.8 mm to (118.5, 183.4)
- moved C56 229.0 mm to (118.5, 171.4)
- moved C64 199.4 mm to (122.9, 165.4)
- moved RV1 158.6 mm to (18.7, 16.3)
- moved R2 132.5 mm to (96.2, 189.4), turned to 0 degrees
- moved R1 130.7 mm to (96.2, 186.4), turned to 0 degrees
- moved U28 130.6 mm to (134.6, 24.4)
- moved R27 118.0 mm to (105.0, 210.0)
- moved R9 115.2 mm to (96.2, 210.0)
- moved R16 108.3 mm to (100.6, 204.1)
- moved R17 108.3 mm to (100.6, 207.1)
- moved R15 108.3 mm to (100.6, 201.2)
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Connections:
- C11 pad 1: Net-(U5-+VOUT) -> Net-(U7-VI)
- C12 pad 1: Net-(U6-+VOUT) -> Net-(U8-VI)
- C20 pad 1: Net-(U10-+VOUT) -> Net-(U12-VI)
- C27 pad 1: Net-(U13-+VOUT) -> Net-(U15-VI)
- C28 pad 1: Net-(U14-+VOUT) -> Net-(U16-VI)
- C37 pad 1: Net-(U17-+VOUT) -> Net-(U21-VI)
- C38 pad 1: Net-(U18-+VOUT) -> Net-(U22-VI)
- C39 pad 1: Net-(U19-+VOUT) -> Net-(U23-VI)
- C40 pad 1: Net-(U20-+VOUT) -> Net-(U24-VI)
- C53 pad 1: Net-(U25-+VOUT) -> Net-(U27-VI)
- C54 pad 1: Net-(U26-+VOUT) -> Net-(U30-VI)
- C55 pad 1: Net-(U27-+VOUT) -> Net-(U29-VI)
- C56 pad 1: Net-(U28-+VOUT) -> Net-(U31-VI)
- C56 pad 2: Net-(U28--VOUT) -> CTREF
- C57 pad 1: Net-(U29-GND) -> Net-(U27-GND)
- C59 pad 1: Net-(U31-GND) -> Net-(U29-GND)
- C6 pad 1: Net-(U2-+VOUT) -> Net-(U4-VI)
- C60 pad 1: Net-(U32-GND) -> Net-(U31-GND)
- C60 pad 2: Net-(U28--VOUT) -> CTREF
- C64 pad 2: Net-(U28--VOUT) -> CTREF
- R1 pad 1: Net-(U1-VI) -> Net-(PS13-+Vout)
- R1 pad 2: CT12 -> Net-(U1-VI)
- R10 pad 1: Net-(U10-+VOUT) -> Net-(PS8-+Vout)
- R10 pad 2: CT6 -> Net-(U12-VI)
- R13 pad 1: Net-(U13-+VOUT) -> Net-(U15-VI)
- R13 pad 2: CT5 -> Net-(PS7-+Vout)
- R14 pad 1: Net-(U14-+VOUT) -> Net-(U16-VI)
- R14 pad 2: CT4 -> Net-(PS6-+Vout)
- R17 pad 1: Net-(U17-+VOUT) -> Net-(PS12-+Vout)
- R17 pad 2: CT11 -> Net-(U21-VI)
- R18 pad 1: Net-(U18-+VOUT) -> Net-(PS11-+Vout)
- R18 pad 2: CT10 -> Net-(U22-VI)
- R19 pad 1: Net-(U19-+VOUT) -> Net-(PS10-+Vout)
- R19 pad 2: CT9 -> Net-(U23-VI)
- R20 pad 1: Net-(U20-+VOUT) -> Net-(PS9-+Vout)
- R20 pad 2: CT8 -> Net-(U24-VI)
- R25 pad 1: Net-(U25-+VOUT) -> Net-(U27-VI)
- R25 pad 2: CT3 -> Net-(PS5-+Vout)
- R26 pad 1: Net-(U26-+VOUT) -> Net-(U30-VI)
- R26 pad 2: CT2 -> Net-(PS4-+Vout)
- R27 pad 1: Net-(U27-+VOUT) -> Net-(U29-VI)
- R27 pad 2: CT1 -> Net-(PS2-+Vout)
- R28 pad 1: Net-(U28-+VOUT) -> CTREF
- R28 pad 2: Net-(U28--VOUT) -> CTREF
- R29 pad 2: Net-(U29-GND) -> Net-(U27-GND)
- R3 pad 1: Net-(U2-+VOUT) -> Net-(PS14-+Vout)
- R3 pad 2: CT13 -> Net-(U4-VI)
- R31 pad 2: Net-(U31-GND) -> Net-(U29-GND)
- R32 pad 1: CT1 -> TERMN+
- R32 pad 2: Net-(U32-GND) -> Net-(U31-VI)
- R5 pad 1: Net-(U5-+VOUT) -> Net-(PS16-+Vout)
- R5 pad 2: CT15 -> Net-(U7-VI)
- R6 pad 1: Net-(U6-+VOUT) -> Net-(PS15-+Vout)
- R6 pad 2: CT14 -> Net-(U8-VI)
- R9 pad 1: Net-(U11-VI) -> Net-(PS17-+Vout)
- R9 pad 2: CT7 -> Net-(U11-VI)
- RV1 pad 1: Net-(U1-GND) -> Net-(R47-Pad2)
- RV10 pad 1: Net-(U22-GND) -> Net-(R49-Pad2)
- RV11 pad 1: Net-(U23-GND) -> Net-(R50-Pad2)
- RV12 pad 1: Net-(U24-GND) -> Net-(R51-Pad2)
- RV13 pad 1: Net-(U29-GND) -> Net-(R35-Pad2)
- RV14 pad 1: Net-(U30-GND) -> Net-(R41-Pad2)
- RV15 pad 1: Net-(U31-GND) -> Net-(R36-Pad2)
- RV16 pad 1: Net-(U32-GND) -> Net-(R38-Pad2)
- RV16 pad 2: Net-(U28--VOUT) -> CTREF
- RV16 pad 3: Net-(U28--VOUT) -> CTREF
- RV17 pad 1: Net-(U32-GND) -> unconnected-(RV17-Pad1)
- RV17 pad 2: Net-(U28--VOUT) -> unconnected-(RV17-Pad2)
- RV17 pad 3: Net-(U28--VOUT) -> unconnected-(RV17-Pad3)
- RV2 pad 1: Net-(U4-GND) -> Net-(R46-Pad2)
- RV3 pad 1: Net-(U7-GND) -> Net-(R33-Pad2)
- RV3 pad 2: CT15 -> CT4
- RV3 pad 3: CT15 -> CT4
- RV4 pad 1: Net-(U8-GND) -> Net-(R45-Pad2)
- RV5 pad 1: Net-(U11-GND) -> Net-(R34-Pad2)
- RV5 pad 2: CT7 -> CT5
- RV5 pad 3: CT7 -> CT5
- RV6 pad 1: Net-(U12-GND) -> Net-(R42-Pad2)
- RV7 pad 1: Net-(U15-GND) -> Net-(R43-Pad2)
- RV7 pad 2: CT5 -> CT7
- RV7 pad 3: CT5 -> CT7
- RV8 pad 1: Net-(U16-GND) -> Net-(R44-Pad2)
- RV8 pad 2: CT4 -> CT15
- RV8 pad 3: CT4 -> CT15
- RV9 pad 1: Net-(U21-GND) -> Net-(R48-Pad2)
- U10 pad 4: Net-(U10-+VOUT) -> Net-(PS4-+Vout)
- U10 pad 6: CT6 -> CT2
- U12 pad 3: Net-(U10-+VOUT) -> Net-(U12-VI)
- U13 pad 4: Net-(U13-+VOUT) -> Net-(PS5-+Vout)
- U13 pad 6: CT5 -> CT3
- U14 pad 4: Net-(U14-+VOUT) -> Net-(PS6-+Vout)
- U15 pad 3: Net-(U13-+VOUT) -> Net-(U15-VI)
- U16 pad 3: Net-(U14-+VOUT) -> Net-(U16-VI)
- U17 pad 4: Net-(U17-+VOUT) -> Net-(PS13-+Vout)
- U17 pad 6: CT11 -> CT12
- U18 pad 4: Net-(U18-+VOUT) -> Net-(PS14-+Vout)
- U18 pad 6: CT10 -> CT13
- U19 pad 4: Net-(U19-+VOUT) -> Net-(PS15-+Vout)
- U19 pad 6: CT9 -> CT14
- U2 pad 4: Net-(U2-+VOUT) -> Net-(PS9-+Vout)
- U2 pad 6: CT13 -> CT8
- U20 pad 4: Net-(U20-+VOUT) -> Net-(PS16-+Vout)
- U20 pad 6: CT8 -> CT15
- U21 pad 3: Net-(U17-+VOUT) -> Net-(U21-VI)
- U22 pad 3: Net-(U18-+VOUT) -> Net-(U22-VI)
- U23 pad 3: Net-(U19-+VOUT) -> Net-(U23-VI)
- U24 pad 3: Net-(U20-+VOUT) -> Net-(U24-VI)
- U25 pad 4: Net-(U25-+VOUT) -> Net-(PS7-+Vout)
- U25 pad 6: CT3 -> CT5
- U26 pad 4: Net-(U26-+VOUT) -> Net-(PS8-+Vout)
- U26 pad 6: CT2 -> CT6
- U27 pad 1: GND -> Net-(U27-GND)
- U27 pad 2: 12V -> CT4
- U28 pad 4: Net-(U28-+VOUT) -> TERMN+
- U28 pad 6: Net-(U28--VOUT) -> CTREF
- U29 pad 2: CT4 -> CT2
- U29 pad 3: Net-(U25-+VOUT) -> Net-(U29-VI)
- U3 pad 4: Net-(U1-VI) -> Net-(PS10-+Vout)
- U3 pad 6: CT12 -> CT9
- U30 pad 3: Net-(U26-+VOUT) -> Net-(U30-VI)
- U31 pad 2: CT2 -> CT1
- U31 pad 3: Net-(U27-+VOUT) -> Net-(U31-VI)
- U4 pad 3: Net-(U2-+VOUT) -> Net-(U4-VI)
- U5 pad 4: Net-(U5-+VOUT) -> Net-(PS11-+Vout)
- U5 pad 6: CT15 -> CT10
- U6 pad 4: Net-(U6-+VOUT) -> Net-(PS12-+Vout)
- U6 pad 6: CT14 -> CT11
- U7 pad 3: Net-(U5-+VOUT) -> Net-(U7-VI)
- U8 pad 3: Net-(U6-+VOUT) -> Net-(U8-VI)

Commit message: Backup
Parts:
- added D1: LED, LED_THT:LED_D3.0mm, F.Cu at (-27.6, 106.7)
- added D2: D_Schottky, Resistor_SMD:R_1206_3216Metric, F.Cu at (-18.9, 106.7)
- added F1: Fuse, Resistor_SMD:R_1206_3216Metric, F.Cu at (265.2, 119.4)
- added F2: Fuse, Resistor_SMD:R_1206_3216Metric, F.Cu at (-18.9, 101.6)
- added J1: Barrel_Jack_MountingPin, Connector_Molex:Molex_KK-396_5273-02A_1x02_P3.96mm_Vertical, F.Cu at (262.7, 129.5)
- added J2: Barrel_Jack_MountingPin, Connector_Molex:Molex_KK-396_5273-02A_1x02_P3.96mm_Vertical, F.Cu at (247.5, 129.5)
- added J3: Conn_01x16, Connector_PinHeader_2.54mm:PinHeader_1x16_P2.54mm_Vertical, F.Cu at (264.2, 33.0)
- added J4: Conn_01x08, Connector_PinHeader_2.54mm:PinHeader_1x08_P2.54mm_Vertical, F.Cu at (264.2, 81.3)
- added J5: Barrel_2.0mmPin_PJ064, Connector_BarrelJack:BarrelJack_GCT_DCJ200-10-A_Horizontal, F.Cu at (-26.7, 86.4)
- added RV19: R_Potentiometer_US, Potentiometer_THT:Potentiometer_Alps_RK09Y11_Single_Horizontal, F.Cu at (206.5, 76.0)
- added RV20: R_Potentiometer_US, Potentiometer_THT:Potentiometer_Alps_RK09Y11_Single_Horizontal, F.Cu at (194.4, 76.0)
- added RV21: R_Potentiometer_US, Potentiometer_THT:Potentiometer_Alps_RK09Y11_Single_Horizontal, F.Cu at (62.0, 76.3)
- added RV22: R_Potentiometer_US, Potentiometer_THT:Potentiometer_Alps_RK09Y11_Single_Horizontal, F.Cu at (85.6, 76.0)
- added RV23: R_Potentiometer_US, Potentiometer_THT:Potentiometer_Alps_RK09Y11_Single_Horizontal, F.Cu at (109.8, 76.0)
- added RV24: R_Potentiometer_US, Potentiometer_THT:Potentiometer_Alps_RK09Y11_Single_Horizontal, F.Cu at (121.9, 76.2)
- added RV25: R_Potentiometer_US, Potentiometer_THT:Potentiometer_Alps_RK09Y11_Single_Horizontal, F.Cu at (73.4, 76.1)
- added RV26: R_Potentiometer_US, Potentiometer_THT:Potentiometer_Alps_RK09Y11_Single_Horizontal, F.Cu at (49.8, 76.7)
- added RV27: R_Potentiometer_US, Potentiometer_THT:Potentiometer_Alps_RK09Y11_Single_Horizontal, F.Cu at (37.2, 76.7)
- added RV28: R_Potentiometer_US, Potentiometer_THT:Potentiometer_Alps_RK09Y11_Single_Horizontal, F.Cu at (134.0, 76.0)
- added RV29: R_Potentiometer_US, Potentiometer_THT:Potentiometer_Alps_RK09Y11_Single_Horizontal, F.Cu at (146.1, 76.0)
- added RV30: R_Potentiometer_US, Potentiometer_THT:Potentiometer_Alps_RK09Y11_Single_Horizontal, F.Cu at (158.2, 76.0)
- added RV31: R_Potentiometer_US, Potentiometer_THT:Potentiometer_Alps_RK09Y11_Single_Horizontal, F.Cu at (170.3, 76.0)
- added RV32: R_Potentiometer_US, Potentiometer_THT:Potentiometer_Alps_RK09Y11_Single_Horizontal, F.Cu at (182.4, 76.0)
- added RV33: R_Potentiometer_US, Potentiometer_THT:Potentiometer_Alps_RK09Y11_Single_Horizontal, F.Cu at (98.1, 76.0)
- added RV34: R_Potentiometer_US, Potentiometer_THT:Potentiometer_Alps_RK09Y11_Single_Horizontal, F.Cu at (230.8, 76.0)
- U1, U11, U12, U15, U16, U21, U22, U23, U24, U27, U29, U30, U31, U35, U4, U7, U8: moved to B.Cu
- moved C1 262.5 mm to (338.7, 55.8)
- moved C10 262.5 mm to (338.7, 82.9)
- moved C2 262.5 mm to (338.7, 58.8)
- moved C21 262.5 mm to (347.6, 55.8)
- moved C22 262.5 mm to (347.6, 58.8)
- moved C23 262.5 mm to (347.6, 61.8)
- moved C24 262.5 mm to (347.6, 64.9)
- moved C25 262.5 mm to (347.6, 67.9)
- moved C26 262.5 mm to (347.6, 70.9)
- moved C27 262.5 mm to (347.6, 73.9)
- moved C28 262.5 mm to (347.6, 76.9)
- moved C29 262.5 mm to (347.6, 79.9)
- moved C3 262.5 mm to (338.7, 61.8)
- moved C30 262.5 mm to (347.6, 82.9)
- moved C31 262.5 mm to (352.1, 55.8)
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Connections:
- RV17 pad 1: unconnected-(RV17-Pad1) -> Net-(R38-Pad2)
- RV17 pad 2: unconnected-(RV17-Pad2) -> CTREF
- RV17 pad 3: unconnected-(RV17-Pad3) -> CTREF

Commit message: Schematics are finished.
Need refactoring
Parts:
- moved F1 358.3 mm to (-50.8, -49.3), turned to -90 degrees
- moved C52 348.6 mm to (15.4, 12.4), turned to -90 degrees
- moved J1 338.9 mm to (-41.4, -20.0), turned to -90 degrees
- moved C51 332.9 mm to (30.9, 12.4), turned to -90 degrees
- moved RV18 325.5 mm to (0.78, -110.3), turned to -90 degrees
- moved C50 318.0 mm to (46.4, 12.4), turned to -90 degrees
- moved C60 316.7 mm to (58.4, 176.4), turned to -90 degrees
- moved C69 316.6 mm to (67.4, 180.9), turned to -90 degrees
- moved R28 315.8 mm to (0.00, 49.9), turned to -90 degrees
- moved C67 314.8 mm to (70.4, 180.9), turned to -90 degrees
- moved C59 314.7 mm to (61.4, 176.4), turned to -90 degrees
- moved C58 312.8 mm to (64.4, 176.4), turned to -90 degrees
- moved C64 311.4 mm to (76.4, 180.9), turned to -90 degrees
- moved C57 311.0 mm to (67.4, 176.4), turned to -90 degrees
- moved C63 309.8 mm to (79.4, 180.9), turned to -90 degrees
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